Commit message: added infrared sensors to urdf model and rviz config

File: urdf/xiaomi_gen1.urdf (robot description, URDF)
Before this commit: robot xiaomi_gen1, 5 links, 4 joints
Links:
- added link cliff_sensor_fl_link
- added link cliff_sensor_fr_link
- added link cliff_sensor_l_link
- added link cliff_sensor_r_link
- added link wall_distance_link
Joints:
- added joint cliff_sensor_fl_joint: type fixed, parent base_footprint, child cliff_sensor_fl_link, origin xyz=0.15515 0.04654 0 rpy=0 1.5708 0.174533, axis 0 0 0
- added joint cliff_sensor_fr_joint: type fixed, parent base_footprint, child cliff_sensor_fr_link, origin xyz=0.15515 -0.04654 0 rpy=0 1.5708 -0.174533, axis 0 0 0
- added joint cliff_sensor_l_joint: type fixed, parent base_footprint, child cliff_sensor_l_link, origin xyz=0.06119 0.1499 0 rpy=0 1.5708 1.39626, axis 0 0 0
- added joint cliff_sensor_r_joint: type fixed, parent base_footprint, child cliff_sensor_r_link, origin xyz=0.06119 -0.1499 0 rpy=0 1.5708 -1.39626, axis 0 0 0
- added joint wall_distance_joint: type fixed, parent base_link, child wall_distance_link, origin xyz=0.03918 -0.16021 0 rpy=0 0 -1.11701, axis 0 0 0
